File: robo_crawler_board.kicad_pcb (KiCad board)
At the start: 2 copper layers, 100 x 77.5 mm, 26 parts, among them J1 Screw_Terminal_01x02, J2 Screw_Terminal_01x02, J3 Screw_Terminal_01x02, J4 Screw_Terminal_01x02, J5 Screw_Terminal_01x02, J6 Screw_Terminal_01x02, J7 Screw_Terminal_01x02, U4 DRV8871DDA, U5 DRV8871DDA, U6 DRV8871DDA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

Commit message: saving progress
Parts:
- removed J4, J5, J6, J7: Screw_Terminal_01x02, TerminalBlock:TerminalBlock_bornier-2_P5.08mm
- removed R3, R4, R5, R6: 15k, Resistor_SMD:R_0805_2012Metric
- removed U2: ~, deadzone_footprints:LM2596 DC-DC Buck Converter
- removed U6, U7, U8, U9: DRV8871DDA, Package_SO:Texas_HTSOP-8-1EP_3.9x4.9mm_P1.27mm_EP2.95x4.9mm_Mask2.4x3.1mm_ThermalVias
- H1, H2, H3, H4: value M2 -> MountingHole
- moved J2 112.6 mm to (179.1, 139.7), turned to 0 degrees
- moved U4 104.4 mm to (136.5, 165.1), turned to 0 degrees
- moved R2 64.8 mm to (55.8, 102.6)
- moved U5 44.8 mm to (71.7, 111.7), turned to 0 degrees
- moved R1 41.7 mm to (152.2, 64.4)
- moved U3 37.3 mm to (122.7, 103.3)
- moved J3 29.2 mm to (68.0, 90.5), turned to 0 degrees
- moved U1 25.4 mm to (125.3, 77.6)
- moved H1 24.4 mm to (66.0, 48.3)
- moved H3 23.3 mm to (205.7, 128.3)
- moved J1 21.5 mm to (163.8, 106.7), turned to 0 degrees
- moved H4 20.8 mm to (74.9, 139.7)
- moved H2 20.3 mm to (201.9, 61.0)
Connections:
- net Net-(J1-Pin_2) renamed +18V
- J1 pad 1: Net-(J1-Pin_1) -> GND
- U1 pad 11: MOTOR6_CH1 -> MOTOR2_CH1
- U1 pad 12: MOTOR6_CH2 -> MOTOR2_CH2
- U1 pad 13: MOTOR2_CH1 -> unconnected-(U1-IO14-Pad13)
- U1 pad 14: MOTOR1_CH1 -> unconnected-(U1-IO12-Pad14)
- U1 pad 16: MOTOR1_CH2 -> unconnected-(U1-IO13-Pad16)
- U1 pad 25: MOTOR2_CH2 -> unconnected-(U1-IO0-Pad25)
- U1 pad 27: MOTOR3_CH1 -> unconnected-(U1-IO16-Pad27)
- U1 pad 28: MOTOR3_CH2 -> unconnected-(U1-IO17-Pad28)
- U1 pad 30: MOTOR4_CH1 -> DRIVE_CH1
- U1 pad 31: MOTOR4_CH2 -> DRIVE_CH2
- U1 pad 36: MOTOR5_CH1 -> MOTOR1_CH1
- U1 pad 37: MOTOR5_CH2 -> MOTOR1_CH2
- U3 pad 1: Net-(J1-Pin_1) -> GND
Routing:
- net +12V: track 135.4 -> 0.00 mm, vias 6 -> 0
- net +5V: track 117.0 -> 0.00 mm
- net MOTOR4_CH2: track 60.7 -> 0.00 mm, vias 1 -> 0
- net GND: track 59.3 -> 0.00 mm, vias 3 -> 0
- net MOTOR5_CH2: track 57.9 -> 0.00 mm, vias 1 -> 0
- net +18V: track 57.8 -> 0.00 mm
- net Net-(J1-Pin_1): track 57.1 -> 0.00 mm
- net MOTOR4_CH1: track 53.3 -> 0.00 mm, vias 1 -> 0
- net MOTOR5_CH1: track 52.9 -> 0.00 mm, vias 1 -> 0
- net MOTOR2_CH2: track 45.7 -> 0.00 mm, vias 1 -> 0
- net MOTOR1_CH1: track 41.4 -> 0.00 mm, vias 1 -> 0
- net MOTOR3_CH2: track 40.0 -> 0.00 mm, vias 1 -> 0
- net MOTOR2_CH1: track 38.7 -> 0.00 mm, vias 1 -> 0
- net MOTOR3_CH1: track 37.0 -> 0.00 mm, vias 1 -> 0
- net MOTOR1_CH2: track 36.4 -> 0.00 mm, vias 1 -> 0
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- removed copper zone on B.Cu, net GND
- removed copper zone on F.Cu, net GND
Other:
- board outline removed
- board text removed: "IN+"
- board text removed: "IN-"
